Commit message: Add proximity sensors to URDF

File: prox2f_description/urdf/prox2f.urdf.xacro (robot description, xacro)
@@ -28,9 +28,40 @@
         <origin xyz="0 0 0" rpy="0 0 ${pi}" />
     </joint>
+    <!-- Frames for proximity sensors -->
+    <xacro:macro name="proximity_frame" params="name parent">
+        <link name="${name}" />
+        <joint name="${name}_joint" type="fixed">
+            <parent link="${parent}" />
+            <child link="${name}" />
+            <origin xyz="-3.5013e-3 0 29e-3" rpy="0 -${pi/2} 0" />
+        </joint>
+        <!-- Create dummy link for gazebo_ros_camera because it publishes image in wrong orientation -->
+        <xacro:if value="$(arg sim_gazebo)">
+            <link name="${name}_gazebo" />
+            <joint name="${name}_gazebo_joint" type="fixed">
+                <parent link="${name}" />
+                <child link="${name}_gazebo" />
+                <origin xyz="0 0 0" rpy="0 -${pi/2} ${pi/2}" />
+            </joint>
+        </xacro:if>
+    </xacro:macro>
+    <xacro:proximity_frame name="left_proximity" parent="robotiq_2f_left_fingertip_link" />
+    <xacro:proximity_frame name="right_proximity" parent="robotiq_2f_right_fingertip_link" />
     <!-- Gazebo -->
-    <gazebo>
-        <plugin filename="libgazebo_ros2_control.so" name="gazebo_ros2_control">
-            <parameters>$(arg simulation_controllers)</parameters>
-        </plugin>
-    </gazebo>
+    <xacro:if value="$(arg sim_gazebo)">
+        <!-- ros2_control -->
+        <gazebo>
+            <plugin filename="libgazebo_ros2_control.so" name="gazebo_ros2_control">
+                <parameters>$(arg simulation_controllers)</parameters>
+            </plugin>
+        </gazebo>
+        <!-- Proximity sensors -->
+        <xacro:include filename="$(find prox2f_description)/urdf/vl53l5cx_macro.xacro" />
+        <gazebo reference="left_proximity_gazebo">
+            <xacro:vl53l5cx name="left_vl53l5cx" frame="left_proximity" />
+        </gazebo>
+        <gazebo reference="right_proximity_gazebo">
+            <xacro:vl53l5cx name="right_vl53l5cx" frame="right_proximity" />
+        </gazebo>
+    </xacro:if>
 </robot>

Commit message: Allow to configure UR initial positions
Add config file for initial positions
Update CmakeLists.txt

File: prox2f_description/urdf/prox2f.urdf.xacro (robot description, xacro)
@@ -8,4 +8,5 @@
     <link name="world" />
     <xacro:include filename="$(find ur_description)/urdf/ur_macro.xacro" />
+    <xacro:property name="initial_positions_file" default="$(find prox2f_description)/config/ur_initial_positions.yaml" />
     <xacro:ur_robot
         name="ur"
@@ -16,4 +17,5 @@
         physical_parameters_file="$(find ur_description)/config/$(arg ur_type)/physical_parameters.yaml"
         visual_parameters_file="$(find ur_description)/config/$(arg ur_type)/visual_parameters.yaml"
+        initial_positions="${xacro.load_yaml(initial_positions_file)}"
         sim_gazebo="$(arg sim_gazebo)"
     >

Commit message: Disable mimic in simulation

File: prox2f_description/urdf/prox2f.urdf.xacro (robot description, xacro)
@@ -5,4 +5,5 @@
     <xacro:arg name="sim_gazebo" default="false" />
     <xacro:arg name="simulation_controllers" default="" />
+    <xacro:property name="sim_gazebo" value="$(arg sim_gazebo)" />
     <!-- UR -->
     <link name="world" />
@@ -24,5 +25,5 @@
     <!-- Gripper -->
     <xacro:include filename="$(find robotiq_2f_85_description)/urdf/robotiq_2f_85_macro.xacro" />
-    <xacro:robotiq_2f_85 name="robotiq_2f" prefix="robotiq_2f_" ur_coupling="true" />
+    <xacro:robotiq_2f_85 name="robotiq_2f" prefix="robotiq_2f_" ur_coupling="true" mimic="${not sim_gazebo}" />
     <joint name="tool_joint" type="fixed">
         <parent link="tool0" />

Commit message: Update TCP position
The z-component of the TCP is slightly larger than the one of the sensor
frame, allowing the gripper to be pushed in the z-direction.

File: prox2f_description/urdf/prox2f.urdf.xacro (robot description, xacro)
@@ -89,5 +89,5 @@
     <parent link="tool0" />
     <child link="tcp" />
-    <origin xyz="0 0 0.15" rpy="0 0 0" />
+    <origin xyz="0 0 0.155" rpy="0 0 0" />
   </joint>
   <!-- Gazebo -->

Commit message: Add frames for attraction center

File: prox2f_description/urdf/prox2f.urdf.xacro (robot description, xacro)
@@ -91,4 +91,17 @@
     <origin xyz="0 0 0.155" rpy="0 0 0" />
   </joint>
+  <!-- Frames for attraction center -->
+  <link name="left_attraction" />
+  <link name="right_attraction" />
+  <joint name="left_attraction_joint" type="fixed">
+    <parent link="tcp" />
+    <child link="left_attraction" />
+    <origin xyz="-0.04 0 0" rpy="0 0 0" />
+  </joint>
+  <joint name="right_attraction_joint" type="fixed">
+    <parent link="tcp" />
+    <child link="right_attraction" />
+    <origin xyz="0.04 0 0" rpy="0 0 0" />
+  </joint>
   <!-- Gazebo -->
   <xacro:if value="$(arg sim_gazebo)">

Commit message: Update sensor frame
For using VL53L7CX.

File: prox2f_description/urdf/prox2f.urdf.xacro (robot description, xacro)
@@ -70,5 +70,5 @@
       <parent link="${parent}" />
       <child link="${name}" />
-      <origin xyz="-3.5013e-3 0 29e-3" rpy="0 -${pi/2} 0" />
+      <origin xyz="-4.25e-3 0 29.51e-3" rpy="0 -${pi/2} 0" />
     </joint>
     <!-- Create dummy link for gazebo_ros_camera because it publishes image in wrong orientation -->

Commit message: Remove attraction frames

File: prox2f_description/urdf/prox2f.urdf.xacro (robot description, xacro)
@@ -91,17 +91,4 @@
     <origin xyz="0 0 0.155" rpy="0 0 0" />
   </joint>
-  <!-- Frames for attraction center -->
-  <link name="left_attraction" />
-  <link name="right_attraction" />
-  <joint name="left_attraction_joint" type="fixed">
-    <parent link="tcp" />
-    <child link="left_attraction" />
-    <origin xyz="-0.04 0 0" rpy="0 0 0" />
-  </joint>
-  <joint name="right_attraction_joint" type="fixed">
-    <parent link="tcp" />
-    <child link="right_attraction" />
-    <origin xyz="0.04 0 0" rpy="0 0 0" />
-  </joint>
   <!-- Gazebo -->
   <xacro:if value="$(arg sim_gazebo)">

Commit message: Update URDF

File: prox2f_description/urdf/prox2f.urdf.xacro (robot description, xacro)
@@ -7,4 +7,5 @@
   <xacro:arg name="simulation_controllers" default="" />
   <xacro:property name="sim_gazebo" value="$(arg sim_gazebo)" />
+  <xacro:arg name="tool_baud_rate" default="1000000" />
   <!-- Gripper parameters -->
   <xacro:arg name="gripper_prefix" default="grp_" />
@@ -13,4 +14,5 @@
   <xacro:arg name="robot_ip" default="0.0.0.0" />
   <xacro:arg name="safety_limits" default="true" />
+  <xacro:arg name="use_tool_communication" default="true" />
   <xacro:arg name="joint_limit_params"
     default="$(find ur_description)/config/$(arg ur_type)/joint_limits.yaml" />
@@ -45,4 +47,7 @@
     sim_gazebo="$(arg sim_gazebo)"
     initial_positions="${xacro.load_yaml(initial_positions_file)}"
+    use_tool_communication="$(arg use_tool_communication)"
+    tool_voltage="12"
+    tool_baud_rate="$(arg tool_baud_rate)"
     robot_ip="$(arg robot_ip)"
     script_filename="$(arg script_filename)"
@@ -53,13 +58,15 @@
   </xacro:ur_robot>
   <!-- Gripper -->
-  <xacro:include filename="$(find robotiq_2f_85_description)/urdf/robotiq_2f_85_macro.xacro" />
-  <xacro:robotiq_2f_85
-    name="grp"
-    prefix="$(arg gripper_prefix)"
-    ur_coupling="true"
-    mimic="${not sim_gazebo}" />
-  <joint name="$(arg gripper_prefix)coupling_joint" type="fixed">
+  <xacro:include filename="$(find e2f_description)/urdf/e2f_macro.xacro" />
+  <xacro:e2f
+    name="e2f"
+    tf_prefix="$(arg gripper_prefix)"
+    use_fake_hardware="$(arg use_fake_hardware)"
+    device_name="/tmp/ttyUR"
+    baud_rate="$(arg tool_baud_rate)"
+  />
+  <joint name="$(arg gripper_prefix)base_joint" type="fixed">
     <parent link="tool0" />
-    <child link="$(arg gripper_prefix)coupling_link" />
+    <child link="$(arg gripper_prefix)base_link" />
     <origin xyz="0 0 0" rpy="0 0 ${pi}" />
   </joint>
@@ -70,5 +77,5 @@
       <parent link="${parent}" />
       <child link="${name}" />
-      <origin xyz="-4.25e-3 0 29.51e-3" rpy="0 -${pi/2} 0" />
+      <origin xyz="-1e-3 0 -9e-3" rpy="-${pi/2} 0 -${pi/2}" />
     </joint>
     <!-- Create dummy link for gazebo_ros_camera because it publishes image in wrong orientation -->
@@ -82,6 +89,6 @@
     </xacro:if>
   </xacro:macro>
-  <xacro:proximity_frame name="left_proximity" parent="$(arg gripper_prefix)left_fingertip_link" />
-  <xacro:proximity_frame name="right_proximity" parent="$(arg gripper_prefix)right_fingertip_link" />
+  <xacro:proximity_frame name="left_proximity" parent="$(arg gripper_prefix)fingertip_l" />
+  <xacro:proximity_frame name="right_proximity" parent="$(arg gripper_prefix)fingertip_r" />
   <!-- Frame for TCP -->
   <link name="tcp" />
@@ -89,5 +96,5 @@
     <parent link="tool0" />
     <child link="tcp" />
-    <origin xyz="0 0 0.155" rpy="0 0 0" />
+    <origin xyz="0 0 0.132" rpy="0 0 0" />
   </joint>
   <!-- Gazebo -->

Commit message: Add workspace collision

File: prox2f_description/urdf/prox2f.urdf.xacro (robot description, xacro)
@@ -54,5 +54,5 @@
     input_recipe_filename="$(arg input_recipe_filename)"
   >
-    <origin xyz="0 0 0" rpy="0 0 0" />
+    <origin xyz="0 0 0" rpy="0 0 ${-pi/2}" />
   </xacro:ur_robot>
   <!-- Gripper -->
@@ -97,4 +97,10 @@
     <origin xyz="0 0 0.132" rpy="0 0 0" />
   </joint>
+  <!-- Workspace -->
+  <xacro:include filename="$(find prox2f_description)/urdf/workspace_macro.xacro" />
+  <xacro:workspace name="workspace" frame="world"
+    size_x="1.1" size_y="0.9" size_z="1.0"
+    center_x="0.15" center_y="0.0" center_z="0.5"
+  />
   <!-- Gazebo -->
   <xacro:if value="$(arg sim_gazebo)">

Commit message: Add aruco marker frame for workspace

File: prox2f_description/urdf/prox2f.urdf.xacro (robot description, xacro)
@@ -103,4 +103,10 @@
     center_x="0.15" center_y="0.0" center_z="0.5"
   />
+  <link name="aruco0" />
+  <joint name="aruco0_joint" type="fixed">
+    <parent link="world" />
+    <child link="aruco0" />
+    <origin xyz="0.4 0 0" rpy="0 0 ${pi/2}" />
+  </joint>
   <!-- Gazebo -->
   <xacro:if value="$(arg sim_gazebo)">

Commit message: Attach camera to robot; no need to estimate camera transform

File: prox2f_description/urdf/prox2f.urdf.xacro (robot description, xacro)
@@ -103,10 +103,9 @@
     center_x="0.15" center_y="0.0" center_z="${0.5 + 0.04}"
   />
-  <link name="aruco0" />
-  <joint name="aruco0_joint" type="fixed">
-    <parent link="world" />
-    <child link="aruco0" />
-    <origin xyz="0.4 0 0" rpy="0 0 ${pi/2}" />
-  </joint>
+  <!-- RealSense -->
+  <xacro:include filename="$(find realsense2_description)/urdf/_d435.urdf.xacro" />
+  <xacro:sensor_d435 parent="tool0">
+    <origin xyz="0 -0.0425 0.01815" rpy="${pi/2} -${pi/2} 0" />
+  </xacro:sensor_d435>
   <!-- Gazebo -->
   <xacro:if value="$(arg sim_gazebo)">

Commit message: Fix TCP rotation

File: prox2f_description/urdf/prox2f.urdf.xacro (robot description, xacro)
@@ -95,5 +95,5 @@
     <parent link="tool0" />
     <child link="tcp" />
-    <origin xyz="0 0 0.132" rpy="0 0 0" />
+    <origin xyz="0 0 0.132" rpy="0 0 ${pi}" />
   </joint>
   <!-- Workspace -->
